Commit message: reconnect WSL project

File: kinematic_utils/cr7_robot_right.urdf (robot description, URDF)
Before this commit: robot cr7_robot, 25 links, 24 joints
Links:
- link Link1: geometry collision mesh filename=cr7_speed/J1.STL; visual mesh filename=cr7_speed/J1.STL
- link Link2: geometry collision mesh filename=cr7_speed/J2.STL; visual mesh filename=cr7_speed/J2.STL
- link Link3: geometry collision mesh filename=cr7_speed/J3.STL; visual mesh filename=cr7_speed/J3.STL
- link Link4: geometry collision mesh filename=cr7_speed/J4.STL; visual mesh filename=cr7_speed/J4.STL
- link Link5: geometry collision mesh filename=cr7_speed/J5.STL; visual mesh filename=cr7_speed/J5.STL
- link Link6: geometry collision mesh filename=cr7_speed/J6.STL; visual mesh filename=cr7_speed/J6.STL
- link RFF_joint1_link: geometry collision mesh filename=cr7_speed/RFF_joint1_link.STL; visual mesh filename=cr7_speed/RFF_joint1_link.STL
- link RFF_joint2_link: geometry collision mesh filename=cr7_speed/RFF_joint2_link.STL; visual mesh filename=cr7_speed/RFF_joint2_link.STL
- link RFF_joint3_link: geometry collision mesh filename=cr7_speed/RFF_joint3_link.STL; visual mesh filename=cr7_speed/RFF_joint3_link.STL
- link RLF_joint1_link: geometry collision mesh filename=cr7_speed/RLF_joint1_link.STL; visual mesh filename=cr7_speed/RLF_joint1_link.STL
- link RLF_joint2_link: geometry collision mesh filename=cr7_speed/RLF_joint2_link.STL; visual mesh filename=cr7_speed/RLF_joint2_link.STL
- link RLF_joint3_link: geometry collision mesh filename=cr7_speed/RLF_joint3_link.STL; visual mesh filename=cr7_speed/RLF_joint3_link.STL
- link RMF_joint1_link: geometry collision mesh filename=cr7_speed/RMF_joint1_link.STL; visual mesh filename=cr7_speed/RMF_joint1_link.STL
- link RMF_joint2_link: geometry collision mesh filename=cr7_speed/RMF_joint2_link.STL; visual mesh filename=cr7_speed/RMF_joint2_link.STL
- link RMF_joint3_link: geometry collision mesh filename=cr7_speed/RMF_joint3_link.STL; visual mesh filename=cr7_speed/RMF_joint3_link.STL
- link RRF_joint1_link: geometry collision mesh filename=cr7_speed/RRF_joint1_link.STL; visual mesh filename=cr7_speed/RRF_joint1_link.STL
- link RRF_joint2_link: geometry collision mesh filename=cr7_speed/RRF_joint2_link.STL; visual mesh filename=cr7_speed/RRF_joint2_link.STL
- link RRF_joint3_link: geometry collision mesh filename=cr7_speed/RRF_joint3_link.STL; visual mesh filename=cr7_speed/RRF_joint3_link.STL
- link RTh_joint1_link: geometry collision mesh filename=cr7_speed/RTh_joint1_link.STL; visual mesh filename=cr7_speed/RTh_joint1_link.STL
- link RTh_joint2_link: geometry collision mesh filename=cr7_speed/RTh_joint2_link.STL; visual mesh filename=cr7_speed/RTh_joint2_link.STL
- link RTh_joint3_link: geometry collision mesh filename=cr7_speed/RTh_joint3_link.STL; visual mesh filename=cr7_speed/RTh_joint3_link.STL
- link base_link: geometry collision mesh filename=cr7_speed/base_link0.STL; visual mesh filename=cr7_speed/base_link0.STL
- link hand_base_link: geometry collision mesh filename=cr7_speed/hand_base_link.STL; visual mesh filename=cr7_speed/hand_base_link.STL
